File: Mench Reloaded/Mench Reloaded.kicad_pcb (KiCad board)
At the start: 2 copper layers, 160 x 100 mm, 4 parts

Commit message: First draft of PCB
Parts:
- added C1: 47pF, Capacitor_SMD:C_0805_2012Metric_Pad1.18x1.45mm_HandSolder, F.Cu at (110.9, 113.0)
- added C10: 0.1uF, Capacitor_SMD:C_0805_2012Metric_Pad1.18x1.45mm_HandSolder, F.Cu at (67.7, 71.3)
- added C11: 0.1uF, Capacitor_SMD:C_0805_2012Metric_Pad1.18x1.45mm_HandSolder, F.Cu at (154.1, 71.3)
- added C12: 10uF, Capacitor_THT:CP_Radial_D10.0mm_P5.00mm, F.Cu at (77.9, 71.4)
- added C13: 0.1uF, Capacitor_SMD:C_0805_2012Metric_Pad1.18x1.45mm_HandSolder, F.Cu at (159.1, 99.3)
- added C14: 0.1uF, Capacitor_SMD:C_0805_2012Metric_Pad1.18x1.45mm_HandSolder, F.Cu at (116.0, 73.9)
- added C2: 27pF, Capacitor_SMD:C_0805_2012Metric_Pad1.18x1.45mm_HandSolder, F.Cu at (142.9, 94.2)
- added C3: 47pF, Capacitor_SMD:C_0805_2012Metric_Pad1.18x1.45mm_HandSolder, F.Cu at (116.0, 113.0)
- added C4: 47pF, Capacitor_SMD:C_0805_2012Metric_Pad1.18x1.45mm_HandSolder, F.Cu at (142.9, 99.3)
- added C5: 10nF, Capacitor_SMD:C_0805_2012Metric_Pad1.18x1.45mm_HandSolder, F.Cu at (101.8, 106.9)
- added C6: 10nF, Capacitor_SMD:C_0805_2012Metric_Pad1.18x1.45mm_HandSolder, F.Cu at (102.2, 81.5)
- added C7: 100nF, Capacitor_SMD:C_0805_2012Metric_Pad1.18x1.45mm_HandSolder, F.Cu at (118.5, 94.2)
- added C8: 100nF, Capacitor_SMD:C_0805_2012Metric_Pad1.18x1.45mm_HandSolder, F.Cu at (85.5, 94.2)
- added C9: 0.33uF, Capacitor_SMD:C_0805_2012Metric_Pad1.18x1.45mm_HandSolder, F.Cu at (60.1, 71.3)
- added D1: green, LED_SMD:LED_0805_2012Metric_Pad1.15x1.40mm_HandSolder, F.Cu at (150.6, 129.8)
- added D2: green, LED_SMD:LED_0805_2012Metric_Pad1.15x1.40mm_HandSolder, F.Cu at (153.6, 129.8)
- added D3: green, LED_SMD:LED_0805_2012Metric_Pad1.15x1.40mm_HandSolder, F.Cu at (156.6, 129.8)
- added D4: green, LED_SMD:LED_0805_2012Metric_Pad1.15x1.40mm_HandSolder, F.Cu at (159.7, 129.8)
- added D5: green, LED_SMD:LED_0805_2012Metric_Pad1.15x1.40mm_HandSolder, F.Cu at (162.7, 129.8)
- added D6: green, LED_SMD:LED_0805_2012Metric_Pad1.15x1.40mm_HandSolder, F.Cu at (165.8, 129.8)
- added D7: green, LED_SMD:LED_0805_2012Metric_Pad1.15x1.40mm_HandSolder, F.Cu at (168.8, 129.8)
- added D8: green, LED_SMD:LED_0805_2012Metric_Pad1.15x1.40mm_HandSolder, F.Cu at (171.8, 129.8)
- added D9: LED, LED_SMD:LED_0805_2012Metric_Pad1.15x1.40mm_HandSolder, F.Cu at (60.1, 79.0)
- added IC1: DS1813, ds1813_revised:ds1813_revised-TO-92, F.Cu at (62.6, 86.6)
- added J1: FTDI serial, Connector_PinHeader_2.54mm:PinHeader_1x06_P2.54mm_Horizontal, F.Cu at (65.2, 119.6)
- added J2: Conn_01x40_Pin, Connector_PinHeader_2.54mm:PinHeader_1x40_P2.54mm_Vertical, F.Cu at (88.0, 139.9)
- added J3: RAM CSB select, Connector_PinHeader_2.54mm:PinHeader_2x04_P2.54mm_Vertical, F.Cu at (184.5, 63.7)
- added J4: Conn_01x40_Pin, Connector_PinHeader_2.54mm:PinHeader_1x40_P2.54mm_Vertical, F.Cu at (88.0, 51.0)
- added J5: Barrel_Jack_Switch, Connector_BarrelJack:BarrelJack_Horizontal, F.Cu at (68.6, 61.2)
- added R1: 150K, Resistor_SMD:R_0805_2012Metric_Pad1.20x1.40mm_HandSolder, F.Cu at (122.6, 114.5)
- added R10: 3K, Resistor_SMD:R_0805_2012Metric_Pad1.20x1.40mm_HandSolder, F.Cu at (165.9, 134.8)
- added R11: 3K, Resistor_SMD:R_0805_2012Metric_Pad1.20x1.40mm_HandSolder, F.Cu at (168.9, 134.8)
- added R12: 3K, Resistor_SMD:R_0805_2012Metric_Pad1.20x1.40mm_HandSolder, F.Cu at (171.8, 134.8)
- added R13: 3K, Resistor_SMD:R_0805_2012Metric_Pad1.20x1.40mm_HandSolder, F.Cu at (162.7, 66.3)
- added R14: 3K, Resistor_SMD:R_0805_2012Metric_Pad1.20x1.40mm_HandSolder, F.Cu at (67.7, 79.0)
- added R2: 1.5K, Resistor_SMD:R_0805_2012Metric_Pad1.20x1.40mm_HandSolder, F.Cu at (125.1, 99.3)
- added R3: 20M, Resistor_SMD:R_0805_2012Metric_Pad1.20x1.40mm_HandSolder, F.Cu at (122.6, 109.4)
- added R4: 1M, Resistor_SMD:R_0805_2012Metric_Pad1.20x1.40mm_HandSolder, F.Cu at (125.1, 94.2)
- added R5: 3K, Resistor_SMD:R_0805_2012Metric_Pad1.20x1.40mm_HandSolder, F.Cu at (150.3, 134.8)
- added R6: 3K, Resistor_SMD:R_0805_2012Metric_Pad1.20x1.40mm_HandSolder, F.Cu at (153.2, 134.8)
- added R7: 3K, Resistor_SMD:R_0805_2012Metric_Pad1.20x1.40mm_HandSolder, F.Cu at (156.2, 134.8)
- added R8: 3K, Resistor_SMD:R_0805_2012Metric_Pad1.20x1.40mm_HandSolder, F.Cu at (159.1, 134.8)
- added R9: 3K, Resistor_SMD:R_0805_2012Metric_Pad1.20x1.40mm_HandSolder, F.Cu at (163.0, 134.8)
- added RN1: 3K, Resistor_THT:R_Array_SIP6, F.Cu at (75.3, 101.8)
- added SW1: SW_Push, Button_Switch_THT:SW_PUSH_6mm_H5mm, F.Cu at (59.4, 94.5)
- added U1: W65C265SxQ, Package_QFP:PQFP-100_14x20mm_P0.65mm, F.Cu at (101.7, 94.2)
- added U2: 128K RAM, Package_DIP:DIP-32_W15.24mm_Socket_LongPads, F.Cu at (160.4, 86.6)
- added U3: 28C256, Package_DIP:DIP-28_W15.24mm_Socket_LongPads, F.Cu at (165.5, 114.5)
- added U4: LM7805_TO220, Package_TO_SOT_THT:TO-220-3_Vertical, F.Cu at (77.9, 58.6)
- added U5: 74HC00, Package_DIP:DIP-14_W7.62mm_Socket_LongPads, F.Cu at (121.0, 81.5)
- added Y1: 32.768 kHz, Crystal:Crystal_C26-LF_D2.1mm_L6.5mm_Horizontal, F.Cu at (112.5, 117.9)
- added Y2: 3.6864 mHz, Crystal:Crystal_HC49-U_Vertical, F.Cu at (133.9, 94.4)
Routing:
- net +5V: track 0.00 -> 21.3 mm
- net GND: track 0.00 -> 5.94 mm
- net Net-(D4-K): track 0.00 -> 3.25 mm
- net Net-(D3-K): track 0.00 -> 3.22 mm
- net Net-(D2-K): track 0.00 -> 3.18 mm
- net Net-(D5-K): track 0.00 -> 3.14 mm
- net Net-(D1-K): track 0.00 -> 3.14 mm
- net Net-(D6-K): track 0.00 -> 3.10 mm
- net Net-(D7-K): track 0.00 -> 3.07 mm
- net Net-(D8-K): track 0.00 -> 3.03 mm
