File: OP-80A/OP-80A.kicad_pcb (KiCad board)
At the start: 2 copper layers, 100 x 100 mm, 37 parts, among them J1 Conn_02x08_Odd_Even, Q1 H10TB, Q2 H10TB, Q3 H10TB, Q4 H10TB, Q5 H10TB, Q6 H10TB, Q7 H10TB, Q8 H10TB, Q9 H10TB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

Commit message: Added external power jack for illumnation lamp. Added trimmer pots to calibrate phototransistors,
Parts:
- added J2: Illumination Power Jack, TerminalBlock_4Ucon:TerminalBlock_4Ucon_1x02_P3.50mm_Horizontal, F.Cu at (89.7, 57.7)
- added REF**: M5, MountingHole:MountingHole_2.2mm_M2, F.Cu at (75.0, 115.0)
- added REF**: M6, MountingHole:MountingHole_2.2mm_M2, F.Cu at (75.0, 144.8)
- added REF**: M8, MountingHole:MountingHole_2.2mm_M2, F.Cu at (125.0, 144.8)
- added REF**: M7, MountingHole:MountingHole_2.2mm_M2, F.Cu at (125.0, 115.0)
- added RV1: 10K, Potentiometer_THT:Potentiometer_Runtron_RM-065_Vertical, F.Cu at (58.2, 107.7)
- added RV2: 10K, Potentiometer_THT:Potentiometer_Runtron_RM-065_Vertical, F.Cu at (68.1, 107.7)
- added RV3: 10K, Potentiometer_THT:Potentiometer_Runtron_RM-065_Vertical, F.Cu at (78.0, 107.7)
- added RV4: 10K, Potentiometer_THT:Potentiometer_Runtron_RM-065_Vertical, F.Cu at (87.9, 107.7)
- added RV5: 10K, Potentiometer_THT:Potentiometer_Runtron_RM-065_Vertical, F.Cu at (97.8, 107.7)
- added RV6: 10K, Potentiometer_THT:Potentiometer_Runtron_RM-065_Vertical, F.Cu at (108.0, 107.7)
- added RV7: 10K, Potentiometer_THT:Potentiometer_Runtron_RM-065_Vertical, F.Cu at (118.1, 107.7)
- added RV8: 10K, Potentiometer_THT:Potentiometer_Runtron_RM-065_Vertical, F.Cu at (128.3, 107.7)
- added RV9: 10K, Potentiometer_THT:Potentiometer_Runtron_RM-065_Vertical, F.Cu at (138.3, 107.7)
- J1: value Conn_02x08_Odd_Even -> Data and power connector
- RN1: value 25K -> 20K
- moved RN1 31.2 mm to (57.7, 97.3)
- moved U10 5.59 mm to (130.0, 88.5)
- moved U3 5.59 mm to (59.3, 88.4)
- moved U4 5.59 mm to (69.3, 88.4)
- moved U5 5.59 mm to (79.5, 88.4)
- moved U6 5.59 mm to (89.5, 88.3)
- moved U7 5.59 mm to (99.7, 88.4)
- moved U8 5.59 mm to (109.9, 88.4)
- moved U9 5.59 mm to (119.9, 88.4)
- moved U11 5.59 mm to (140.1, 88.6)
- moved SW1 3.05 mm to (104.4, 57.9)
- moved Q5 0.83 mm to (100.4, 129.5)
- moved Q1 0.83 mm to (100.3, 119.4)
- moved Q2 0.83 mm to (100.3, 121.9)
- moved Q3 0.83 mm to (100.3, 124.5)
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- renumbered D2 to D1, D3 to D2, D1 to D3
Connections:
- RN1 pad 10: Net-(Q9-C) -> Net-(RN1-R9)
- RN1 pad 2: Net-(Q1-C) -> Net-(RN1-R1)
- RN1 pad 3: Net-(Q2-C) -> Net-(RN1-R2)
- RN1 pad 4: Net-(Q3-C) -> Net-(RN1-R3)
- RN1 pad 5: Net-(Q4-C) -> Net-(RN1-R4)
- RN1 pad 6: Net-(Q5-C) -> Net-(RN1-R5)
- RN1 pad 7: Net-(Q6-C) -> Net-(RN1-R6)
- RN1 pad 8: Net-(Q7-C) -> Net-(RN1-R7)
- RN1 pad 9: Net-(Q8-C) -> Net-(RN1-R8)
Routing:
- net Net-(RN1-R9): track 0.00 -> 66.0 mm, vias 0 -> 1
- net Net-(RN1-R8): track 0.00 -> 58.3 mm, vias 0 -> 1
- net Net-(RN1-R7): track 0.00 -> 50.3 mm, vias 0 -> 1
- net +5V: track 398.4 -> 349.0 mm, vias 31 -> 32
- net Net-(RN1-R6): track 0.00 -> 42.3 mm, vias 0 -> 1
- net Net-(RN1-R5): track 0.00 -> 35.0 mm, vias 0 -> 1
- net Net-(RN1-R4): track 0.00 -> 27.3 mm, vias 0 -> 1
- net GND: track 372.9 -> 395.4 mm, vias 15 -> 16
- net Net-(RN1-R3): track 0.00 -> 19.4 mm, vias 0 -> 1
- net Net-(D4-A): track 167.4 -> 153.7 mm
- net Net-(Q9-C): track 78.8 -> 91.7 mm
- net Net-(RN1-R2): track 0.00 -> 12.6 mm
- net Net-(RN1-R1): track 0.00 -> 11.2 mm
- net Net-(Q8-C): track 71.4 -> 79.7 mm
- net Net-(Q6-C): track 47.6 -> 55.1 mm
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