File: OP-80A/OP-80A.kicad_sch (KiCad schematic)
At the start: 33 parts, among them J1 Conn_02x08_Odd_Even, Q1 BPW42, Q2 BPW42, Q3 BPW42, Q4 BPW42, Q5 BPW42, Q6 BPW42, Q7 BPW42, Q8 BPW42, Q9 BPW42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

Commit message: First draft of board and routing.
Parts:
- C1, C2: footprint (none) -> Capacitor_THT:C_Disc_D3.0mm_W1.6mm_P2.50mm
- D1: renamed from D2; footprint (none) -> LED_THT:LED_D5.0mm
- D2: renamed from D1; footprint (none) -> LED_THT:LED_D5.0mm
- D3, D4: footprint (none) -> LED_THT:LED_D5.0mm
- J1: footprint (none) -> Connector_PinSocket_2.54mm:PinSocket_2x08_P2.54mm_Vertical
- Q1, Q2, Q3, Q4, Q5, Q6, Q7, Q8, Q9: value BPW42 -> H10TB; footprint LED_THT:LED_D3.0mm_Clear -> LED_SMD:LED_0805_2012Metric_Pad1.15x1.40mm_HandSolder
- R1: renamed from R3; footprint (none) -> Resistor_THT:R_Axial_DIN0204_L3.6mm_D1.6mm_P7.62mm_Horizontal
- R2: footprint (none) -> Resistor_THT:R_Axial_DIN0204_L3.6mm_D1.6mm_P7.62mm_Horizontal
- R3: renamed from R4; footprint (none) -> Resistor_THT:R_Axial_DIN0204_L3.6mm_D1.6mm_P7.62mm_Horizontal
- R4: renamed from R1; footprint (none) -> Resistor_THT:R_Axial_DIN0204_L3.6mm_D1.6mm_P7.62mm_Horizontal
- SW1: footprint (none) -> Button_Switch_THT:SW_Slide-03_Wuerth-WS-SLTV_10x2.5x6.4_P2.54mm
- U1: renamed from U5; footprint (none) -> Package_SO:SO-14_5.3x10.2mm_P1.27mm
- U2: renamed from U3; footprint (none) -> Package_SO:SO-14_5.3x10.2mm_P1.27mm
- renumbered U1 to U3, U2 to U4, U4 to U5

Commit message: Added external power jack for illumnation lamp. Added trimmer pots to calibrate phototransistors,
Parts:
- added J2: Illumination Power Jack, TerminalBlock_4Ucon:TerminalBlock_4Ucon_1x02_P3.50mm_Horizontal, symbol Connector_Generic:Conn_01x02
- added RV1, RV2, RV3, RV4, RV5, RV6, RV7, RV8, RV9: 10K, Potentiometer_THT:Potentiometer_Runtron_RM-065_Vertical, symbol Device:R_Potentiometer_Trim_US
- J1: value Conn_02x08_Odd_Even -> Data and power connector
- RN1: value 25K -> 20K
- renumbered D2 to D1, D3 to D2, D1 to D3
Connections:
- net +5V: now also J2.1 (Pin_1)
- net GND: now also J2.2 (Pin_2)
- net at Q7.1 (C), U9.2 (TR), U9.6 (THR): now also RV7.2; no longer RN1.8 (R7)
- net at Q4.1 (C), U6.2 (TR), U6.6 (THR): now also RV4.2; no longer RN1.5 (R4)
- net at Q8.1 (C), U10.2 (TR), U10.6 (THR): now also RV8.2; no longer RN1.9 (R8)
- net at Q9.1 (C), U11.2 (TR), U11.6 (THR): now also RV9.2; no longer RN1.10 (R9)
- net at Q1.1 (C), U3.2 (TR), U3.6 (THR): now also RV1.2; no longer RN1.2 (R1)
- net at Q2.1 (C), U4.2 (TR), U4.6 (THR): now also RV2.2; no longer RN1.3 (R2)
- net at Q3.1 (C), U5.2 (TR), U5.6 (THR): now also RV3.2; no longer RN1.4 (R3)
- net at Q5.1 (C), U7.2 (TR), U7.6 (THR): now also RV5.2; no longer RN1.6 (R5)
- net at Q6.1 (C), U8.2 (TR), U8.6 (THR): now also RV6.2; no longer RN1.7 (R6)
- new net: RN1.6 (R5), RV5.1
- new net: RN1.10 (R9), RV9.1
- new net: RN1.4 (R3), RV3.1
- new net: RN1.2 (R1), RV1.1
- new net: RN1.3 (R2), RV2.1
- new net: RN1.5 (R4), RV4.1
- new net: RN1.7 (R6), RV6.1
- new net: RN1.8 (R7), RV7.1
- new net: RN1.9 (R8), RV8.1
Other:
- moved on the sheet: C1, C2, D2, D3, Q1, Q2, Q3, Q4, Q5, Q6, Q7, Q8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
