File: RiSC-16/noodling.kicad_sch (KiCad schematic)
At the start: 10 parts, among them U23 74LS151, U24 74LS151, U25 74LS373, U26 74LS373, U27 74LS373, U28 74LS373, U29 74LS373, U30 74LS373, U31 74LS373, U32 74LS137

Commit message: Check point of design.
Parts:
- renumbered U23 to U26, U24 to U27, U25 to U28, U26 to U29, U27 to U30, U28 to U31, U29 to U32, U30 to U33, U31 to U34, U32 to U35
Changed lines of the file:
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@@
 		(dnp no)
 		(fields_autoplaced yes)
-		(property "Reference" "#PWR063"
+		(property "Reference" "#PWR069"
 			(at 116.84 171.45 0)
 			(effects
@@
 			(project ""
 				(path "/09ce4153-429f-4803-b069-3af485a81dd6/3a113de7-a305-4b13-86ca-d80a92ced471"
-					(reference "#PWR063")
+					(reference "#PWR069")
 					(unit 1)
 				)
@@
 		(dnp no)
 		(fields_autoplaced yes)
-		(property "Reference" "#PWR060"
+		(property "Reference" "#PWR066"
 			(at 187.96 143.51 0)
 			(effects
@@
 			(project "RiSC-16"
 				(path "/09ce4153-429f-4803-b069-3af485a81dd6/3a113de7-a305-4b13-86ca-d80a92ced471"
-					(reference "#PWR060")
+					(reference "#PWR066")
 					(unit 1)
 				)
@@
 		(dnp no)
 		(fields_autoplaced yes)
-		(property "Reference" "#PWR049"
+		(property "Reference" "#PWR055"
 			(at 119.38 31.75 0)
 			(effects
@@
 			(project ""
 				(path "/09ce4153-429f-4803-b069-3af485a81dd6/3a113de7-a305-4b13-86ca-d80a92ced471"
-					(reference "#PWR049")
+					(reference "#PWR055")
 					(unit 1)
 				)
@@
 		(dnp no)
 		(fields_autoplaced yes)
-		(property "Reference" "#PWR051"
+		(property "Reference" "#PWR057"
 			(at 100.33 35.56 0)
 			(effects
@@
 			(project "RiSC-16"
 				(path "/09ce4153-429f-4803-b069-3af485a81dd6/3a113de7-a305-4b13-86ca-d80a92ced471"
-					(reference "#PWR051")
+					(reference "#PWR057")
 					(unit 1)
 				)
@@
 		(dnp no)
 		(fields_autoplaced yes)
-		(property "Reference" "#PWR059"
+		(property "Reference" "#PWR065"
 			(at 148.59 143.51 0)
 			(effects
@@
 			(project "RiSC-16"
 				(path "/09ce4153-429f-4803-b069-3af485a81dd6/3a113de7-a305-4b13-86ca-d80a92ced471"
-					(reference "#PWR059")
+					(reference "#PWR065")
 					(unit 1)
 				)
@@
 		(dnp no)
 		(fields_autoplaced yes)
-		(property "Reference" "U28"
+		(property "Reference" "U31"
 			(at 150.7333 97.79 0)
 			(effects
@@
 			(project "RiSC-16"
 				(path "/09ce4153-429f-4803-b069-3af485a81dd6/3a113de7-a305-4b13-86ca-d80a92ced471"
-					(reference "U28")
+					(reference "U31")
 					(unit 1)
 				)
@@
 		(dnp no)
 		(fields_autoplaced yes)
-		(property "Reference" "#PWR057"
+		(property "Reference" "#PWR063"
 			(at 71.12 143.51 0)
 			(effects
@@
 			(project "RiSC-16"
 				(path "/09ce4153-429f-4803-b069-3af485a81dd6/3a113de7-a305-4b13-86ca-d80a92ced471"
-					(reference "#PWR057")
+					(reference "#PWR063")
 					(unit 1)
 				)
@@
 		(dnp no)
 		(fields_autoplaced yes)
-		(property "Reference" "U26"
+		(property "Reference" "U29"
 			(at 73.2633 97.79 0)
 			(effects
@@
 			(project "RiSC-16"
 				(path "/09ce4153-429f-4803-b069-3af485a81dd6/3a113de7-a305-4b13-86ca-d80a92ced471"
-					(reference "U26")
+					(reference "U29")
 					(unit 1)
 				)
@@
 		(dnp no)
 		(fields_autoplaced yes)
-		(property "Reference" "#PWR053"
+		(property "Reference" "#PWR059"
 			(at 119.38 82.55 0)
 			(effects
@@
 			(project ""
 				(path "/09ce4153-429f-4803-b069-3af485a81dd6/3a113de7-a305-4b13-86ca-d80a92ced471"
-					(reference "#PWR053")
+					(reference "#PWR059")
 					(unit 1)
 				)
@@
 		(dnp no)
 		(fields_autoplaced yes)
-		(property "Reference" "U24"
+		(property "Reference" "U27"
 			(at 188.8333 27.94 0)
 			(effects
@@
 			(project ""
 				(path "/09ce4153-429f-4803-b069-3af485a81dd6/3a113de7-a305-4b13-86ca-d80a92ced471"
-					(reference "U24")
+					(reference "U27")
 					(unit 1)
 				)
@@
 		(dnp no)
 		(fields_autoplaced yes)
-		(property "Reference" "U32"
+		(property "Reference" "U35"
 			(at 156.21 169.3067 0)
 			(effects
@@
 			(project ""
 				(path "/09ce4153-429f-4803-b069-3af485a81dd6/3a113de7-a305-4b13-86ca-d80a92ced471"
-					(reference "U32")
+					(reference "U35")
 					(unit 1)
 				)
@@
 		(dnp no)
 		(fields_autoplaced yes)
-		(property "Reference" "U31"
+		(property "Reference" "U34"
 			(at 268.8433 96.52 0)
 			(effects
@@
 			(project "RiSC-16"
 				(path "/09ce4153-429f-4803-b069-3af485a81dd6/3a113de7-a305-4b13-86ca-d80a92ced471"
-					(reference "U31")
+					(reference "U34")
 					(unit 1)
 				)
@@
 		(dnp no)
 		(fields_autoplaced yes)
-		(property "Reference" "#PWR056"
+		(property "Reference" "#PWR062"
 			(at 33.02 143.51 0)
 			(effects
@@
 			(project "RiSC-16"
 				(path "/09ce4153-429f-4803-b069-3af485a81dd6/3a113de7-a305-4b13-86ca-d80a92ced471"
-					(reference "#PWR056")
+					(reference "#PWR062")
 					(unit 1)
 				)
@@
 		(dnp no)
 		(fields_autoplaced yes)
-		(property "Reference" "U23"
+		(property "Reference" "U26"
 			(at 121.5233 27.94 0)
 			(effects
@@
 			(project "RiSC-16"
 				(path "/09ce4153-429f-4803-b069-3af485a81dd6/3a113de7-a305-4b13-86ca-d80a92ced471"
-					(reference "U23")
+					(reference "U26")
 					(unit 1)
 				)
@@
 		(dnp no)
 		(fields_autoplaced yes)
-		(property "Reference" "#PWR064"
+		(property "Reference" "#PWR070"
 			(at 152.4 171.45 0)
 			(effects
@@
 			(project ""
 				(path "/09ce4153-429f-4803-b069-3af485a81dd6/3a113de7-a305-4b13-86ca-d80a92ced471"
-					(reference "#PWR064")
+					(reference "#PWR070")
 					(unit 1)
 				)
@@
 		(dnp no)
 		(fields_autoplaced yes)
-		(property "Reference" "#PWR052"
+		(property "Reference" "#PWR058"
 			(at 167.64 35.56 0)
 			(effects
@@
 			(project "RiSC-16"
 				(path "/09ce4153-429f-4803-b069-3af485a81dd6/3a113de7-a305-4b13-86ca-d80a92ced471"
-					(reference "#PWR052")
+					(reference "#PWR058")
 					(unit 1)
 				)
@@
 		(dnp no)
 		(fields_autoplaced yes)
-		(property "Reference" "#PWR054"
+		(property "Reference" "#PWR060"
 			(at 186.69 82.55 0)
 			(effects
@@
 			(project ""
 				(path "/09ce4153-429f-4803-b069-3af485a81dd6/3a113de7-a305-4b13-86ca-d80a92ced471"
-					(reference "#PWR054")
+					(reference "#PWR060")
 					(unit 1)
 				)
@@
 		(dnp no)
 		(fields_autoplaced yes)
-		(property "Reference" "U30"
+		(property "Reference" "U33"
 			(at 228.2033 96.52 0)
 			(effects
@@
 			(project "RiSC-16"
 				(path "/09ce4153-429f-4803-b069-3af485a81dd6/3a113de7-a305-4b13-86ca-d80a92ced471"
-					(reference "U30")
+					(reference "U33")
 					(unit 1)
 				)
@@
 		(dnp no)
 		(fields_autoplaced yes)
-		(property "Reference" "#PWR058"
+		(property "Reference" "#PWR064"
 			(at 109.22 143.51 0)
 			(effects
@@
 			(project "RiSC-16"
 				(path "/09ce4153-429f-4803-b069-3af485a81dd6/3a113de7-a305-4b13-86ca-d80a92ced471"
-					(reference "#PWR058")
+					(reference "#PWR064")
 					(unit 1)
 				)
@@
 		(dnp no)
 		(fields_autoplaced yes)
-		(property "Reference" "U25"
+		(property "Reference" "U28"
 			(at 35.1633 97.79 0)
 			(effects
@@
 			(project ""
 				(path "/09ce4153-429f-4803-b069-3af485a81dd6/3a113de7-a305-4b13-86ca-d80a92ced471"
-					(reference "U25")
+					(reference "U28")
 					(unit 1)
 				)
@@
 		(dnp no)
 		(fields_autoplaced yes)
-		(property "Reference" "#PWR062"
+		(property "Reference" "#PWR068"
 			(at 266.7 143.51 0)
 			(effects
@@
 			(project "RiSC-16"
 				(path "/09ce4153-429f-4803-b069-3af485a81dd6/3a113de7-a305-4b13-86ca-d80a92ced471"
-					(reference "#PWR062")
+					(reference "#PWR068")
 					(unit 1)
 				)
@@
 		(dnp no)
 		(fields_autoplaced yes)
-		(property "Reference" "#PWR050"
+		(property "Reference" "#PWR056"
 			(at 186.69 31.75 0)
 			(effects
@@
 			(project ""
 				(path "/09ce4153-429f-4803-b069-3af485a81dd6/3a113de7-a305-4b13-86ca-d80a92ced471"
-					(reference "#PWR050")
+					(reference "#PWR056")
 					(unit 1)
 				)
@@
 		(dnp no)
 		(fields_autoplaced yes)
-		(property "Reference" "#PWR061"
+		(property "Reference" "#PWR067"
 			(at 226.06 143.51 0)
 			(effects
@@
 			(project "RiSC-16"
 				(path "/09ce4153-429f-4803-b069-3af485a81dd6/3a113de7-a305-4b13-86ca-d80a92ced471"
-					(reference "#PWR061")
+					(reference "#PWR067")
 					(unit 1)
 				)
@@
 		(dnp no)
 		(fields_autoplaced yes)
-		(property "Reference" "U27"
+		(property "Reference" "U30"
 			(at 111.3633 97.79 0)
 			(effects
@@
 			(project "RiSC-16"
 				(path "/09ce4153-429f-4803-b069-3af485a81dd6/3a113de7-a305-4b13-86ca-d80a92ced471"
-					(reference "U27")
+					(reference "U30")
 					(unit 1)
 				)
@@
 		(dnp no)
 		(fields_autoplaced yes)
-		(property "Reference" "U29"
+		(property "Reference" "U32"
 			(at 190.1033 96.52 0)
 			(effects
@@
 			(project "RiSC-16"
 				(path "/09ce4153-429f-4803-b069-3af485a81dd6/3a113de7-a305-4b13-86ca-d80a92ced471"
-					(reference "U29")
+					(reference "U32")
 					(unit 1)
 				)
@@
 		(dnp no)
 		(fields_autoplaced yes)
-		(property "Reference" "#PWR055"
+		(property "Reference" "#PWR061"
 			(at 33.02 100.33 0)
 			(effects
@@
 			(project ""
 				(path "/09ce4153-429f-4803-b069-3af485a81dd6/3a113de7-a305-4b13-86ca-d80a92ced471"
-					(reference "#PWR055")
-					(unit 1)
-				)
+					(reference "#PWR061")
+					(unit 1)
+				)

Commit message: Annotated the schematic to align part numbers. EPROM and RAM board was added last revision. Reworked the src1 latching to assert 0xf to select the PC.
Parts:
- renumbered U26 to U27, U27 to U28, U28 to U29, U29 to U30, U30 to U31, U31 to U32, U32 to U33, U33 to U34, U34 to U35, U35 to U36
Changed lines of the file:
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@@
 		(dnp no)
 		(fields_autoplaced yes)
-		(property "Reference" "#PWR069"
+		(property "Reference" "#PWR066"
 			(at 116.84 171.45 0)
 			(effects
@@
 			(project ""
 				(path "/09ce4153-429f-4803-b069-3af485a81dd6/3a113de7-a305-4b13-86ca-d80a92ced471"
-					(reference "#PWR069")
+					(reference "#PWR066")
 					(unit 1)
 				)
@@
 		(dnp no)
 		(fields_autoplaced yes)
-		(property "Reference" "#PWR066"
+		(property "Reference" "#PWR063"
 			(at 187.96 143.51 0)
 			(effects
@@
 			(project "RiSC-16"
 				(path "/09ce4153-429f-4803-b069-3af485a81dd6/3a113de7-a305-4b13-86ca-d80a92ced471"
-					(reference "#PWR066")
+					(reference "#PWR063")
 					(unit 1)
 				)
@@
 		(dnp no)
 		(fields_autoplaced yes)
-		(property "Reference" "#PWR055"
+		(property "Reference" "#PWR052"
 			(at 119.38 31.75 0)
 			(effects
@@
 			(project ""
 				(path "/09ce4153-429f-4803-b069-3af485a81dd6/3a113de7-a305-4b13-86ca-d80a92ced471"
-					(reference "#PWR055")
+					(reference "#PWR052")
 					(unit 1)
 				)
@@
 		(dnp no)
 		(fields_autoplaced yes)
-		(property "Reference" "#PWR057"
+		(property "Reference" "#PWR054"
 			(at 100.33 35.56 0)
 			(effects
@@
 			(project "RiSC-16"
 				(path "/09ce4153-429f-4803-b069-3af485a81dd6/3a113de7-a305-4b13-86ca-d80a92ced471"
-					(reference "#PWR057")
+					(reference "#PWR054")
 					(unit 1)
 				)
@@
 		(dnp no)
 		(fields_autoplaced yes)
-		(property "Reference" "#PWR065"
+		(property "Reference" "#PWR062"
 			(at 148.59 143.51 0)
 			(effects
@@
 			(project "RiSC-16"
 				(path "/09ce4153-429f-4803-b069-3af485a81dd6/3a113de7-a305-4b13-86ca-d80a92ced471"
-					(reference "#PWR065")
+					(reference "#PWR062")
 					(unit 1)
 				)
@@
 		(dnp no)
 		(fields_autoplaced yes)
-		(property "Reference" "U31"
+		(property "Reference" "U32"
 			(at 150.7333 97.79 0)
 			(effects
@@
 			(project "RiSC-16"
 				(path "/09ce4153-429f-4803-b069-3af485a81dd6/3a113de7-a305-4b13-86ca-d80a92ced471"
-					(reference "U31")
+					(reference "U32")
 					(unit 1)
 				)
@@
 		(dnp no)
 		(fields_autoplaced yes)
-		(property "Reference" "#PWR063"
+		(property "Reference" "#PWR060"
 			(at 71.12 143.51 0)
 			(effects
@@
 			(project "RiSC-16"
 				(path "/09ce4153-429f-4803-b069-3af485a81dd6/3a113de7-a305-4b13-86ca-d80a92ced471"
-					(reference "#PWR063")
+					(reference "#PWR060")
 					(unit 1)
 				)
@@
 		(dnp no)
 		(fields_autoplaced yes)
-		(property "Reference" "U29"
+		(property "Reference" "U30"
 			(at 73.2633 97.79 0)
 			(effects
@@
 			(project "RiSC-16"
 				(path "/09ce4153-429f-4803-b069-3af485a81dd6/3a113de7-a305-4b13-86ca-d80a92ced471"
-					(reference "U29")
+					(reference "U30")
 					(unit 1)
 				)
@@
 		(dnp no)
 		(fields_autoplaced yes)
-		(property "Reference" "#PWR059"
+		(property "Reference" "#PWR056"
 			(at 119.38 82.55 0)
 			(effects
@@
 			(project ""
 				(path "/09ce4153-429f-4803-b069-3af485a81dd6/3a113de7-a305-4b13-86ca-d80a92ced471"
-					(reference "#PWR059")
+					(reference "#PWR056")
 					(unit 1)
 				)
@@
 		(dnp no)
 		(fields_autoplaced yes)
-		(property "Reference" "U27"
+		(property "Reference" "U28"
 			(at 188.8333 27.94 0)
 			(effects
@@
 			(project ""
 				(path "/09ce4153-429f-4803-b069-3af485a81dd6/3a113de7-a305-4b13-86ca-d80a92ced471"
-					(reference "U27")
+					(reference "U28")
 					(unit 1)
 				)
@@
 		(dnp no)
 		(fields_autoplaced yes)
-		(property "Reference" "U35"
+		(property "Reference" "U36"
 			(at 156.21 169.3067 0)
 			(effects
@@
 			(project ""
 				(path "/09ce4153-429f-4803-b069-3af485a81dd6/3a113de7-a305-4b13-86ca-d80a92ced471"
-					(reference "U35")
+					(reference "U36")
 					(unit 1)
 				)
@@
 		(dnp no)
 		(fields_autoplaced yes)
-		(property "Reference" "U34"
+		(property "Reference" "U35"
 			(at 268.8433 96.52 0)
 			(effects
@@
 			(project "RiSC-16"
 				(path "/09ce4153-429f-4803-b069-3af485a81dd6/3a113de7-a305-4b13-86ca-d80a92ced471"
-					(reference "U34")
+					(reference "U35")
 					(unit 1)
 				)
@@
 		(dnp no)
 		(fields_autoplaced yes)
-		(property "Reference" "#PWR062"
+		(property "Reference" "#PWR059"
 			(at 33.02 143.51 0)
 			(effects
@@
 			(project "RiSC-16"
 				(path "/09ce4153-429f-4803-b069-3af485a81dd6/3a113de7-a305-4b13-86ca-d80a92ced471"
-					(reference "#PWR062")
+					(reference "#PWR059")
 					(unit 1)
 				)
@@
 		(dnp no)
 		(fields_autoplaced yes)
-		(property "Reference" "U26"
+		(property "Reference" "U27"
 			(at 121.5233 27.94 0)
 			(effects
@@
 			(project "RiSC-16"
 				(path "/09ce4153-429f-4803-b069-3af485a81dd6/3a113de7-a305-4b13-86ca-d80a92ced471"
-					(reference "U26")
+					(reference "U27")
 					(unit 1)
 				)
@@
 		(dnp no)
 		(fields_autoplaced yes)
-		(property "Reference" "#PWR070"
+		(property "Reference" "#PWR067"
 			(at 152.4 171.45 0)
 			(effects
@@
 			(project ""
 				(path "/09ce4153-429f-4803-b069-3af485a81dd6/3a113de7-a305-4b13-86ca-d80a92ced471"
-					(reference "#PWR070")
+					(reference "#PWR067")
 					(unit 1)
 				)
@@
 		(dnp no)
 		(fields_autoplaced yes)
-		(property "Reference" "#PWR058"
+		(property "Reference" "#PWR055"
 			(at 167.64 35.56 0)
 			(effects
@@
 			(project "RiSC-16"
 				(path "/09ce4153-429f-4803-b069-3af485a81dd6/3a113de7-a305-4b13-86ca-d80a92ced471"
-					(reference "#PWR058")
+					(reference "#PWR055")
 					(unit 1)
 				)
@@
 		(dnp no)
 		(fields_autoplaced yes)
-		(property "Reference" "#PWR060"
+		(property "Reference" "#PWR057"
 			(at 186.69 82.55 0)
 			(effects
@@
 			(project ""
 				(path "/09ce4153-429f-4803-b069-3af485a81dd6/3a113de7-a305-4b13-86ca-d80a92ced471"
-					(reference "#PWR060")
+					(reference "#PWR057")
 					(unit 1)
 				)
@@
 		(dnp no)
 		(fields_autoplaced yes)
-		(property "Reference" "U33"
+		(property "Reference" "U34"
 			(at 228.2033 96.52 0)
 			(effects
@@
 			(project "RiSC-16"
 				(path "/09ce4153-429f-4803-b069-3af485a81dd6/3a113de7-a305-4b13-86ca-d80a92ced471"
-					(reference "U33")
+					(reference "U34")
 					(unit 1)
 				)
@@
 		(dnp no)
 		(fields_autoplaced yes)
-		(property "Reference" "#PWR064"
+		(property "Reference" "#PWR061"
 			(at 109.22 143.51 0)
 			(effects
@@
 			(project "RiSC-16"
 				(path "/09ce4153-429f-4803-b069-3af485a81dd6/3a113de7-a305-4b13-86ca-d80a92ced471"
-					(reference "#PWR064")
+					(reference "#PWR061")
 					(unit 1)
 				)
@@
 		(dnp no)
 		(fields_autoplaced yes)
-		(property "Reference" "U28"
+		(property "Reference" "U29"
 			(at 35.1633 97.79 0)
 			(effects
@@
 			(project ""
 				(path "/09ce4153-429f-4803-b069-3af485a81dd6/3a113de7-a305-4b13-86ca-d80a92ced471"
-					(reference "U28")
+					(reference "U29")
 					(unit 1)
 				)
@@
 		(dnp no)
 		(fields_autoplaced yes)
-		(property "Reference" "#PWR068"
+		(property "Reference" "#PWR065"
 			(at 266.7 143.51 0)
 			(effects
@@
 			(project "RiSC-16"
 				(path "/09ce4153-429f-4803-b069-3af485a81dd6/3a113de7-a305-4b13-86ca-d80a92ced471"
-					(reference "#PWR068")
+					(reference "#PWR065")
 					(unit 1)
 				)
@@
 		(dnp no)
 		(fields_autoplaced yes)
-		(property "Reference" "#PWR056"
+		(property "Reference" "#PWR053"
 			(at 186.69 31.75 0)
 			(effects
@@
 			(project ""
 				(path "/09ce4153-429f-4803-b069-3af485a81dd6/3a113de7-a305-4b13-86ca-d80a92ced471"
-					(reference "#PWR056")
+					(reference "#PWR053")
 					(unit 1)
 				)
@@
 		(dnp no)
 		(fields_autoplaced yes)
-		(property "Reference" "#PWR067"
+		(property "Reference" "#PWR064"
 			(at 226.06 143.51 0)
 			(effects
@@
 			(project "RiSC-16"
 				(path "/09ce4153-429f-4803-b069-3af485a81dd6/3a113de7-a305-4b13-86ca-d80a92ced471"
-					(reference "#PWR067")
+					(reference "#PWR064")
 					(unit 1)
 				)
@@
 		(dnp no)
 		(fields_autoplaced yes)
-		(property "Reference" "U30"
+		(property "Reference" "U31"
 			(at 111.3633 97.79 0)
 			(effects
@@
 			(project "RiSC-16"
 				(path "/09ce4153-429f-4803-b069-3af485a81dd6/3a113de7-a305-4b13-86ca-d80a92ced471"
-					(reference "U30")
+					(reference "U31")
 					(unit 1)
 				)
@@
 		(dnp no)
 		(fields_autoplaced yes)
-		(property "Reference" "U32"
+		(property "Reference" "U33"
 			(at 190.1033 96.52 0)
 			(effects
@@
 			(project "RiSC-16"
 				(path "/09ce4153-429f-4803-b069-3af485a81dd6/3a113de7-a305-4b13-86ca-d80a92ced471"
-					(reference "U32")
+					(reference "U33")
 					(unit 1)
 				)
@@
 		(dnp no)
 		(fields_autoplaced yes)
-		(property "Reference" "#PWR061"
+		(property "Reference" "#PWR058"
 			(at 33.02 100.33 0)
 			(effects
@@
 			(project ""
 				(path "/09ce4153-429f-4803-b069-3af485a81dd6/3a113de7-a305-4b13-86ca-d80a92ced471"
-					(reference "#PWR061")
-					(unit 1)
-				)
+					(reference "#PWR058")
+					(unit 1)
+				)
